File: Documentation/Schematics/JOC-SkyVision-Rev.1.09/JOC-SkyVision-Rev.1.09.sch (KiCad schematic (older format))
At the start: 103 parts, among them Q1 KAK (Transistor?), Q2 JAJ (Transistor?), Q3 KAK (Transistor?), U1 AZ1117C-ADJ (GH15E) 5V, U10 ON MC34063A (INVERTING REGULA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, U2 809SL (Reset Supervisor), U3 AZ1117C-ADJ (GH16D) 3.3V, U4 MaxLinear SP232E, U5 AT45DB161E (16M+512K SPI Flas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, U6 LPC2148FBD64, U7 GENITOP GT23L16U2W (FONT/CHAR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, U8 TI (74)LVC07A (OPEN DRAIN HEX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, U9 Speaker_Crystal, X1 Crystal (RTC), X2 Crystal (MCU)

Commit message: updated schematics
Added power stage
Added keypad matrix (MCU connection still missing)
Added LED stage
Updated PC interface
Updated motor interface
Added Display net, missing Connection to MCU
Parts:
- added C18, C19, C20, C21, C22, C23, C24, C25, C26, C27: C, symbol Device:C
- added KEYPAD3, KEYPAD4: SW_DIP_x10, symbol Switch:SW_DIP_x10
- added R28, R29, R30, R51, R59, R6, R60, R7, R8, R9: R, symbol Device:R
- LCD1: value Conn_01x36_Male -> Zero Force Flat Cable Connector
Connections:
- net PWR_VCC is gone; now on net PCISP: F1.1
- net U1_INPUT is gone; now on net U10_5V_OUT: U1.3 (Pin_3), U3.3 (Pin_3)
- net U1_OUTPUT is gone; now on net PCISP: U1.2 (Pin_2)
- net U3_OUTPUT is gone; now on net VCC_3.3V: C17.1, JP3.4 (VDD), Q2.3 (E), R19.2, R24.1, R27.1, R31.2, R32.2, R33.2, R34.2, R35.2, R36.1, R38.2, R50.2, R54.2, R55.2, U3.2 (Pin_2), U5.5 (Pin_5), U5.6 (Pin_6), U6.23 (VDD), U6.43 (VDD), U6.51 (VDD), U6.63 (VREF), U7.7 (Pin_7), U8.14 (Pin_14)
- net U3_VOUT is gone; now on net VCC_3.3V: U3.4 (Pin_4)
- net U8_4A is gone; now on net MCU_P1.22: R50.1, U8.9 (Pin_9)
- net U8_6Y is gone; now on net MCU_P1.21: R33.1, U8.12 (Pin_12)
- net LCD_BG_LED1: now also KEYPADLEDS1.10 (Pin_10), KEYPADLEDS1.2 (Pin_2), KEYPADLEDS1.4 (Pin_4), KEYPADLEDS1.6 (Pin_6), KEYPADLEDS1.8 (Pin_8), KEYPADLEDS2.10 (Pin_10), KEYPADLEDS2.2 (Pin_2), KEYPADLEDS2.4 (Pin_4), KEYPADLEDS2.6 (Pin_6), KEYPADLEDS2.8 (Pin_8)
- net MCU_GND: now also C10.1, LCD1.24 (Pin_24), LCD1.25 (Pin_25), LCD1.26 (Pin_26), LCD1.27 (Pin_27), LCD1.28 (Pin_28), LCD1.29 (Pin_29), LCD1.4 (Pin_4), LCD1.5 (Pin_5), R56.1, C18.1, C21.1, C22.1, C23.1, C24.1, C25.1, C26.1; no longer C10.2
- net MCU_P0.8_TXD1: no longer R34.1, U6.34 (P0.9), U8.6 (Pin_6)
- net MCU_P1.17: now also U6.10 (D+), U6.11 (D-)
- net PCISP: now also C6.1, R37.1, R28.2, R29.2, R30.2, R51.2, R59.2, R6.2, R60.2, R7.2, R8.2, R9.2; no longer U6.41 (P0.14)
- net U10_CMP_INV_IN: now also R39.1, R56.2
- net MCU_P0.21: now reaches U6.1 (P0.21)
- net MCU_P0.21: now also R22.2
- net MCU_P1.31: now reaches U6.20 (P1.31)
- net MCU_P0.2: now reaches U6.22 (P0.2)
- net MCU_P1.26: now reaches U6.24 (P1.26)
- net MCU_P0.3: now reaches U6.26 (P0.3)
- net MCU_P0.7: now reaches U6.31 (P0.7)
- net MCU_P0.10: now reaches U6.35 (P0.10)
- net MCU_P1.23: now reaches U6.36 (P1.23)
- net MCU_P0.11: now reaches U6.37 (P0.11)
- net MCU_P0.12: now reaches U6.38 (P0.12)
- net MCU_P0.13: now reaches U6.39 (P0.13)
- net MCU_P1.22: now reaches U6.40 (P1.22)
- net MCU_P1.21: now reaches U6.44 (P1.21)
- net MCU_P0.15: now reaches U6.45 (P0.15)
- net MCU_P1.30: now reaches U6.52 (P1.30)
- net MCU_P1.29: now reaches U6.56 (P1.29)
- net MCU_P0.23: now reaches U6.58 (P0.23)
- net MCU_P1.28: now reaches U6.60 (P1.28)
- net MCU_P1.27: now reaches U6.64 (P1.27)
- net MCU_P1.18: now reaches U6.8 (P1.18)
- net at D3.1 (K), U10.2 (Pin_2): now also L1.1
- net KEY_COLUMN1: now reaches KEYPAD1.1
- net KEY_COLUMN1: now also KEYPAD1.2, KEYPAD1.3, KEYPAD1.5, KEYPAD1.7
- net KEY_COLUMN3: now reaches KEYPAD1.10
- net KEY_COLUMN3: now also KEYPAD1.8, KEYPAD3.3, KEYPAD3.6, KEYPAD3.9
- net at KEYPAD1.11: now also KEYPAD2.10
- net at KEYPAD1.12: now also KEYPAD2.9
- net at KEYPAD1.13: now also KEYPAD2.8
- net at KEYPAD1.14: now also KEYPAD2.7
- net at KEYPAD1.15: now also KEYPAD2.6
- net at KEYPAD1.16: now also KEYPAD2.5
- net at KEYPAD1.17: now also KEYPAD2.4
- net at KEYPAD1.18: now also KEYPAD2.3
- net at KEYPAD1.19: now also KEYPAD2.2
- net at KEYPAD1.20: now also KEYPAD2.1
- net KEY_COLUMN2: now reaches KEYPAD1.4
- net KEY_COLUMN2: now also KEYPAD1.9, KEYPAD3.2, KEYPAD3.5, KEYPAD3.8
- net KEY_COLUMN4: now reaches KEYPAD1.6
- net KEY_COLUMN4: now also KEYPAD3.1, KEYPAD3.10, KEYPAD3.4, KEYPAD3.7
- net KEY_ENTER_OUT: now reaches KEYPAD2.11
- net KEY_ENTER_OUT: now also KEYPAD2.12, KEYPAD2.14, KEYPAD4.20
- net KEY_DOWN_OUT: now reaches KEYPAD2.13
- net KEY_DOWN_OUT: now also KEYPAD2.15, KEYPAD2.16, KEYPAD2.17
- net KEY_F_OUT: now reaches KEYPAD2.18
- net KEY_F_OUT: now also KEYPAD4.11, KEYPAD4.12, KEYPAD4.13
- net KEY_EIGHT_OUT: now reaches KEYPAD2.19
- net KEY_EIGHT_OUT: now also KEYPAD4.14, KEYPAD4.15, KEYPAD4.16
- net KEY_FIVE_OUT: now reaches KEYPAD2.20
- net KEY_FIVE_OUT: now also KEYPAD4.17, KEYPAD4.18, KEYPAD4.19
- net at KEYPADLEDS1.1 (Pin_1): now also R8.1
- net at KEYPADLEDS1.11 (Pin_11): now also KEYPADLEDS1.12 (Pin_12)
- net at KEYPADLEDS1.13 (Pin_13): now also KEYPADLEDS1.14 (Pin_14)
- net at KEYPADLEDS1.15 (Pin_15): now also KEYPADLEDS1.16 (Pin_16)
- net at KEYPADLEDS1.17 (Pin_17): now also KEYPADLEDS1.18 (Pin_18)
- net at KEYPADLEDS1.19 (Pin_19): now also KEYPADLEDS1.20 (Pin_20)
- net at KEYPADLEDS1.3 (Pin_3): now also R60.1
- net at KEYPADLEDS1.5 (Pin_5): now also R29.1
- net at KEYPADLEDS1.7 (Pin_7): now also R30.1
- net at KEYPADLEDS1.9 (Pin_9): now also R51.1
- net at KEYPADLEDS2.1 (Pin_1): now also R7.1
- net at KEYPADLEDS2.11 (Pin_11): now also KEYPADLEDS2.12 (Pin_12)
- net at KEYPADLEDS2.13 (Pin_13): now also KEYPADLEDS2.14 (Pin_14)
- net at KEYPADLEDS2.15 (Pin_15): now also KEYPADLEDS2.16 (Pin_16)
- net at KEYPADLEDS2.17 (Pin_17): now also KEYPADLEDS2.18 (Pin_18)
- net at KEYPADLEDS2.19 (Pin_19): now also KEYPADLEDS2.20 (Pin_20)
- net at KEYPADLEDS2.3 (Pin_3): now also R59.1
- net at KEYPADLEDS2.5 (Pin_5): now also R9.1
- net at KEYPADLEDS2.7 (Pin_7): now also R6.1
- net at KEYPADLEDS2.9 (Pin_9): now also R28.1
- net LCD_10: now reaches LCD1.10 (Pin_10)
- net LCD_10: now also C22.2
- net LCD_11: now reaches LCD1.11 (Pin_11)
- net LCD_11: now also C25.2
- net LCD_12: now reaches LCD1.12 (Pin_12)
- net LCD_12: now also C18.2
- net LCD_14: now reaches LCD1.14 (Pin_14)
- net LCD_14: now also C27.1
- net LCD_15: now reaches LCD1.15 (Pin_15)
- net LCD_15: now also C27.2
- net LCD_16: now reaches LCD1.16 (Pin_16)
- net LCD_16: now also C19.1
- net LCD_17: now reaches LCD1.17 (Pin_17)
- net LCD_17: now also C19.2, C20.1
- net LCD_18: now reaches LCD1.18 (Pin_18)
- net LCD_18: now also C20.2
- net LCD_19: now reaches LCD1.19 (Pin_19)
- net LCD_19: now also C21.2
- net VCC_3.3V: now reaches LCD1.21 (Pin_21)
- net VCC_3.3V: now also C10.2, LCD1.30 (Pin_30), LCD1.31 (Pin_31), R17.2, R18.2, C24.2
- net LCD_8: now reaches LCD1.8 (Pin_8)
- net LCD_8: now also C23.2
- net LCD_9: now reaches LCD1.9 (Pin_9)
- net LCD_9: now also C26.2
- net MCU_P0.14_ISP: now reaches R37.2
- net MCU_P0.14_ISP: now also U6.41 (P0.14)
- net U10_5V_OUT: now reaches C1.2
- net U10_5V_OUT: now also L1.2, R39.2
- net LED1_3_ENABLE renamed U8_4Y
- new net: KEYPAD3.11, KEYPAD4.10
- new net: KEYPAD3.12, KEYPAD4.9
- new net: KEYPAD3.13, KEYPAD4.8
- new net: KEYPAD3.14, KEYPAD4.7
- new net: KEYPAD3.15, KEYPAD4.6
- new net: KEYPAD3.16, KEYPAD4.5
- new net: KEYPAD3.17, KEYPAD4.4
- new net: KEYPAD3.18, KEYPAD4.3
- new net: KEYPAD3.19, KEYPAD4.2
- new net: KEYPAD3.20, KEYPAD4.1
- new net MCU_P0.9_RXD1: R34.1, U6.34 (P0.9), U8.6 (Pin_6)
- no-connect marks 13 -> 26
Other:
- note added: "F1"
- note added: "KEY COLUMNS"
- note added: "KEY_DOWN"
- note added: "KEY_EIGHT"
- note added: "KEY_ENTER"
- note added: "KEY_F"
- note added: "KEY_FIVE"
- note added: "KEY_FOUR"
- note added: "KEY_HELP"
- note added: "KEY_LEFT"
- note added: "KEY_LIGHT"
- note added: "KEY_MINUS"
- note added: "KEY_NINE"
- note added: "KEY_NULL"
- note added: "KEY_ONE"
- note added: "KEY_PLUS"
- note added: "KEY_RIGHT"
- note added: "KEY_ROWS"
- note added: "KEY_SEVEN"
- note added: "KEY_SIX"
- note added: "KEY_THREE"
- note added: "KEY_TWO"
- note added: "KEY_UP"
- note added: "Keypad Background LED Assembly"
- note added: "Keypad Matrix Assembly"
- note added: "RJ45 HBX to Motors Assembly"
- note added: "This is implemented\nin 5x4 key matrix configuration."
- note added: "Two LEDs are connected in series, \nsharing one series resistor.\nNot aligned to key layout!"
- note removed: "RJ45 Assembly"
- moved on the sheet: BT1, C1, C10, C11, C12, C13, C14, C15, C16, C17, C2, C28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
