File: Documentation/Schematics/JOC-SkyVision-Rev.1.09/JOC-SkyVision-Rev.1.09.sch (KiCad schematic (older format))
At the start: 125 parts, among them Q1 KAK (Transistor?), Q2 JAJ (Transistor?), Q3 KAK (Transistor?), U1 AZ1117C-ADJ (GH15E) 5V, U10 ON MC34063A (INVERTING REGULA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, U2 809SL (Reset Supervisor), U3 AZ1117C-ADJ (GH16D) 3.3V, U4 MaxLinear SP232E, U5 AT45DB161E (16M+512K SPI Flas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, U6 LPC2148FBD64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

Commit message: updated schematic for handbox
Parts:
- added LCD_BG_LED1: LED, symbol Device:LED
Connections:
- net KEY_COLUMN2: no longer R12.1, R13.1, U6.11 (D-)
- net KEY_COLUMN3: now also R2.1
- net LCD_BG_LED1: now also LCD_BG_LED1.1 (K)
- net LCD_BG_LED2: now also LCD_BG_LED1.2 (A)
- net MCU_P0.14_ISP: now also R36.2
- net MCU_P0.18: no longer R2.1
- net USB_D+: now also R13.1
- net VCC_3.3V: now also C11.2, R15.2, R16.2
- net ?: now reaches R10.2
- net ?: now also R1.2, R12.2, R13.2, R14.2, R2.2
- new net USB_D-: R12.1, U6.11 (D-)
Other:
- note added: "LC Display Assembly"
- note added: "MCU and Pullup Resistors"
- moved on the sheet: C11, C15, C16, C18, C19, C2, C20, C21, C22, C23, C24, C25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
