File: Documentation/Schematics/JOC-SkyVision-Handbox-Rev.1.09/JOC-SkyVision-Rev.1.09.sch (KiCad schematic (older format))
At the start: 126 parts, among them Q1 KAK (Transistor?), Q2 JAJ (Transistor?), Q3 KAK (Transistor?), U1 AZ1117C-ADJ (GH15E) 5V, U10 ON MC34063A (INVERTING REGULA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, U2 809SL (Reset Supervisor), U3 AZ1117C-ADJ (GH16D) 3.3V, U4 MaxLinear SP232E, U5 AT45DB161E (16M+512K SPI Flas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, U6 LPC2148FBD64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

Commit message: Fix wrong wiring external interrupt lines for motors
Connections:
- net KEY_ENTER_OUT: no longer R32.1, U8.1 (Pin_1)
- net MCU_P0.7: now also R32.1, U8.1 (Pin_1)
Other:
- note added: "<"
- note added: ">"
Changed lines of the file:
@@
 Text Label 15350 9250 0    50   ~ 0
 MCU_P0.9_RXD1
-Text Label 15350 8850 0    50   ~ 0
-MCU_P0.30
 Wire Wire Line
 	15150 8850 15350 8850
@@
 Text Notes 3750 1450 0    50   ~ 0
 MCU and Pullup Resistors
+Text Label 15350 8850 0    50   ~ 0
+MCU_P0.7
+Text Notes 13450 8900 0    50   ~ 0
+<
+Text Notes 13450 9350 0    50   ~ 0
+>
 $EndSCHEMATC

Commit message: updated schematics
added introduction text for schematics
Other:
- note added: "<OUT HBX"
- note added: "IN HBX>"
- note removed: "<"
- note removed: ">"
- note removed: "INCOMPLETE"
Changed lines of the file:
@@
 U 1 1 62FAB686
 P 13150 9600
-F 0 "D1" H 13300 9550 50  0000 C CNN
+F 0 "D1" H 13150 9500 50  0000 C CNN
 F 1 "D" H 13150 9726 50  0001 C CNN
 F 2 "" H 13150 9600 50  0001 C CNN
@@
 Text Notes 12250 8500 0    50   ~ 0
 RJ45 HBX to Motors Assembly
-Text Notes 15350 10550 0    79   ~ 0
-INCOMPLETE
 Text Label 6300 6950 0    50   ~ 0
 VCC_3.3V
@@
 Text Label 15350 8850 0    50   ~ 0
 MCU_P0.7
-Text Notes 13450 8900 0    50   ~ 0
-<
-Text Notes 13450 9350 0    50   ~ 0
->
+Text Notes 13350 8950 0    50   ~ 0
+<OUT HBX
+Text Notes 13400 9350 0    50   ~ 0
+IN HBX>
 $EndSCHEMATC
